File: sch/pwr.sch (KiCad schematic (older format))
At the start: 0 parts

Commit message: Add voltage regulator
Parts:
- added C21, C22, C23: 10uF, Capacitor_SMD:C_0805_2012Metric, symbol Device:C
- added C24: 4.7uF, Capacitor_SMD:C_0805_2012Metric, symbol Device:C
- added C25, C26: 10nF, Capacitor_SMD:C_0402_1005Metric, symbol Device:C
- added IC7: LT3030IFE#TRPBF, LT3030IFE#TRPBF:SOP65P640X120-21N, symbol LT3030IFE#TRPBF:LT3030IFE#TRPBF
- added R11, R12: 0.1, Resistor_SMD:R_0402_1005Metric, symbol Device:R
- added R13, R14: 100, Resistor_SMD:R_0402_1005Metric, symbol Device:R
- added R15: 357k, Resistor_SMD:R_0402_1005Metric, symbol Device:R
- added R16: 210k, Resistor_SMD:R_0402_1005Metric, symbol Device:R
- added R17, R18: 1M, Resistor_SMD:R_0402_1005Metric, symbol Device:R
Connections:
- new net: IC7.1 (ADJ1), R15.1, R16.2
- new net: C24.2, C26.2, IC7.10 (ADJ2), IC7.7 (OUT2_1), IC7.8 (OUT2_2), R12.1, R13.2
- new net: IC7.12 (PWRGD2), R18.2
- new net: IC7.19 (PWRGD1), R17.2
- new net: C25.1, IC7.2 (BYP1)
- new net: C23.2, C25.2, IC7.3 (OUT1_1), IC7.4 (OUT1_2), R11.1, R14.2, R15.2
- new net: C26.1, IC7.9 (BYP2)
- new net +1V2: C22.2, R12.2
- new net +3V3: C21.2, R11.2
- new net +5V: IC7.11 (~SHDN2), IC7.13 (IN2_1), IC7.14 (IN2_2), IC7.17 (IN1_1), IC7.18 (IN1_2), IC7.20 (~SHDN1), R17.1, R18.1
- new net GND: C21.1, C22.1, C23.1, C24.1, IC7.15 (GND_3), IC7.16 (GND_4), IC7.21 (GND_5), IC7.5 (GND_1), IC7.6 (GND_2), R13.1, R14.1, R16.1
