File: sch/prog.kicad_pcb (KiCad board)
At the start: 2 copper layers, 12 parts, among them IC1 FT2232HQ-TRAY, J1 Conn_01x02_Male, J2 USB3075-30-A, J3 MTMS-105-02-T-D-002, Y1 ECS-5032MV-120-BM-TR

Commit message: Autoroute
Routing:
- net +3V3: track 70.3 -> 106.1 mm, vias 5 -> 2
- net GND: track 96.0 -> 113.6 mm, vias 2 -> 0
- net Net-(C5-Pad1): track 11.6 -> 29.1 mm, vias 3 -> 2
- net SCK: track 33.6 -> 19.5 mm, vias 2 -> 1
- net MOSI: track 31.6 -> 22.8 mm
- net CDONE: track 27.7 -> 35.8 mm, vias 2 -> 0
- net CRESET: track 26.1 -> 32.0 mm, vias 2 -> 0
- net CS: track 18.6 -> 15.8 mm
- net Net-(IC1-Pad6): track 10.5 -> 8.43 mm, vias 2 -> 0
- net +5V: track 14.8 -> 13.5 mm
- net MISO: track 16.4 -> 16.0 mm, vias 2 -> 1
- net Net-(J1-Pad1): track 9.70 -> 9.69 mm, vias 1 -> 0
Other:
- board outline added: 20.6 x 26.2 mm
