File: sch/nhci.kicad_pcb (KiCad board)
At the start: 4 copper layers, 47 x 85.3 mm, 72 parts, among them IC1 74LVC8T245RHLRG4, IC2 74LVC8T245RHLRG4, IC3 74LVC8T245RHLRG4, IC4 74LVC8T245RHLRG4, IC5 74LVC8T245RHLRG4, IC6 MAX3421EEHJ+, IC7 LT3030IFE#TRPBF, J1 CLP-105-02-F-D, SW1 SW_Push_Open, U1 PCMCIA_BOARD, U2 iCE40-HX8K-CT256, U3 N25Q032A13EF440F, U4 LM3526M-H, Y1 ECS-5032MV-120-BM-TR

Commit message: V2.0 board
Parts:
- added IC8: 74LVC8T245RHLRG4, 74LVC8T245RHLRG4:74LVC8T245RHLRG4, B.Cu at (50.0, 109.0)
- JP1: footprint Jumper:SolderJumper-2_P1.3mm_Bridged2Bar_RoundedPad1.0x1.5mm -> Jumper:SolderJumper-2_P1.3mm_Open_RoundedPad1.0x1.5mm
Connections:
- IC1 pad 22: GND -> F_CE1O
- IC6 pad 22: Net-(IC6-Pad22) -> Net-(C29-Pad1)
- U1 pad 37: Net-(U1-Pad37) -> /P_D11
- U1 pad 38: Net-(U1-Pad38) -> /P_D12
- U1 pad 39: Net-(U1-Pad39) -> /P_D13
- U1 pad 40: Net-(U1-Pad40) -> /P_D14
- U1 pad 41: Net-(U1-Pad41) -> /P_D15
- U1 pad 64: Net-(U1-Pad64) -> /P_D8
- U1 pad 65: Net-(U1-Pad65) -> /P_D9
- U1 pad 66: Net-(U1-Pad66) -> /P_D10
- U2 pad N5: Net-(U2-PadN5) -> F_D8
- U2 pad N6: Net-(U2-PadN6) -> F_D14
- U2 pad N7: Net-(U2-PadN7) -> F_D12
- U2 pad P10: Net-(U2-PadP10) -> F_CE1O
- U2 pad P4: Net-(U2-PadP4) -> F_D10
- U2 pad P5: Net-(U2-PadP5) -> F_D9
- U2 pad P6: Net-(U2-PadP6) -> F_D15
- U2 pad P7: Net-(U2-PadP7) -> F_D13
- U2 pad P8: Net-(U2-PadP8) -> F_D11
- U2 pad P9: Net-(U2-PadP9) -> F_CE2O
Routing:
- net /P_D10: track 0.00 -> 42.3 mm, vias 0 -> 1
- net /P_D9: track 0.00 -> 41.2 mm, vias 0 -> 1
- net F_CE2O: track 0.00 -> 40.4 mm, vias 0 -> 3
- net /P_D8: track 0.00 -> 40.3 mm, vias 0 -> 1
- net F_CE1O: track 0.00 -> 36.4 mm, vias 0 -> 2
- net F_D12: track 0.00 -> 26.7 mm, vias 0 -> 1
- net F_D11: track 0.00 -> 26.7 mm, vias 0 -> 1
- net F_D13: track 0.00 -> 24.9 mm, vias 0 -> 1
- net F_D14: track 0.00 -> 24.4 mm, vias 0 -> 1
- net F_D15: track 0.00 -> 22.4 mm, vias 0 -> 1
- net F_D8: track 0.00 -> 21.6 mm, vias 0 -> 1
- net F_D9: track 0.00 -> 20.1 mm, vias 0 -> 1
- net F_D10: track 0.00 -> 18.9 mm, vias 0 -> 1
- net Net-(C29-Pad1): track 61.5 -> 72.5 mm, vias 2 -> 4
- net /P_D15: track 0.00 -> 10.3 mm, vias 0 -> 1
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