File: sch/nhci.sch (KiCad schematic (older format))
At the start: 28 parts, among them IC1 74LVC8T245RHLRG4, IC2 74LVC8T245RHLRG4, IC3 74LVC8T245RHLRG4, IC4 74LVC8T245RHLRG4, IC5 74LVC8T245RHLRG4, SW1 SW_Push_Open, U1 PCMCIA_BOARD

Commit message: V2.0 board
Parts:
- added IC8: 74LVC8T245RHLRG4, 74LVC8T245RHLRG4:74LVC8T245RHLRG4, symbol 74LVC8T245RHLRG4:74LVC8T245RHLRG4
- JP1: footprint Jumper:SolderJumper-2_P1.3mm_Bridged2Bar_RoundedPad1.0x1.5mm -> Jumper:SolderJumper-2_P1.3mm_Open_RoundedPad1.0x1.5mm
Connections:
- net +3V3: now also IC8.1 (VCCA)
- net +5V: now also IC8.23 (VCCB_1), IC8.24 (VCCB_2)
- net F_DDIR: now also IC8.2 (DIR)
- net GND: now also IC8.11 (GND_1), IC8.12 (GND_2), IC8.13 (GND_3); no longer IC1.22 (~OE)
- net P_D11: now reaches U1.37 (D11)
- net P_D11: now also IC8.14 (B8)
- net P_D12: now reaches U1.38 (D12)
- net P_D12: now also IC8.15 (B7)
- net P_D13: now reaches U1.39 (D13)
- net P_D13: now also IC8.16 (B6)
- net P_D14: now reaches U1.40 (D14)
- net P_D14: now also IC8.17 (B5)
- net P_D15: now reaches U1.41 (D15)
- net P_D15: now also IC8.18 (B4)
- net P_D8: now reaches U1.64 (D8)
- net P_D8: now also IC8.19 (B3)
- net P_D9: now reaches U1.65 (D9)
- net P_D9: now also IC8.20 (B2)
- net P_D10: now reaches U1.66 (D10)
- net P_D10: now also IC8.21 (B1)
- new net F_CE1O: IC1.22 (~OE)
- new net F_CE2O: IC8.22 (~OE)
- new net F_D10: IC8.3 (A1)
- new net F_D11: IC8.10 (A8)
- new net F_D12: IC8.9 (A7)
- new net F_D13: IC8.8 (A6)
- new net F_D14: IC8.7 (A5)
- new net F_D15: IC8.6 (A4)
- new net F_D8: IC8.5 (A3)
- new net F_D9: IC8.4 (A2)
Other:
- moved on the sheet: C1, C10, C2, C3, C4, C5, C6, C7, C8, C9
